File: NanoISP.kicad_pcb (KiCad board)
At the start: 2 copper layers, 54 x 40.6 mm, 14 parts, among them J1 Conn_02x03_Odd_Even, J2 Conn_01x02_Male

Commit message: Fixed a small bug.
Connections:
- A1 pad 27: unconnected-(A1-Pad27) -> Net-(A1-Pad27)
- A1 pad 30: Net-(A1-Pad30) -> unconnected-(A1-Pad30)
- J1 pad 2: Net-(A1-Pad30) -> Net-(A1-Pad27)
Routing:
- net /GND: track 33.0 -> 4.60 mm
- net Net-(A1-Pad27): track 0.00 -> 25.2 mm, vias 0 -> 2
- net Net-(A1-Pad30): track 14.3 -> 0.00 mm, vias 2 -> 0
Changed lines of the file:
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@@
   (net 25 "unconnected-(A1-Pad25)")
   (net 26 "unconnected-(A1-Pad26)")
-  (net 27 "unconnected-(A1-Pad27)")
+  (net 27 "Net-(A1-Pad27)")
   (net 28 "Net-(A1-Pad28)")
-  (net 29 "Net-(A1-Pad30)")
+  (net 29 "unconnected-(A1-Pad30)")
   (net 30 "Net-(D1-Pad2)")
   (net 31 "Net-(D2-Pad2)")
@@
       (net 15 "Net-(A1-Pad15)") (pinfunction "Pin_1") (pintype "passive"))
     (pad "2" thru_hole oval (at 2.54 0) (size 1.7 1.7) (drill 1) (layers *.Cu *.Mask)
-      (net 29 "Net-(A1-Pad30)") (pinfunction "Pin_2") (pintype "passive"))
+      (net 27 "Net-(A1-Pad27)") (pinfunction "Pin_2") (pintype "passive"))
     (pad "3" thru_hole oval (at 0 -2.54) (size 1.7 1.7) (drill 1) (layers *.Cu *.Mask)
       (net 16 "Net-(A1-Pad16)") (pinfunction "Pin_3") (pintype "passive"))
@@
       (net 26 "unconnected-(A1-Pad26)") (pinfunction "A7") (pintype "bidirectional+no_connect"))
     (pad "27" thru_hole oval locked (at 15.24 -7.62 270) (size 1.6 1.6) (drill 1) (layers *.Cu *.Mask)
-      (net 27 "unconnected-(A1-Pad27)") (pinfunction "+5V") (pintype "power_out+no_connect"))
+      (net 27 "Net-(A1-Pad27)") (pinfunction "+5V") (pintype "power_out"))
     (pad "28" thru_hole oval locked (at 15.24 -5.08 270) (size 1.6 1.6) (drill 1) (layers *.Cu *.Mask)
       (net 28 "Net-(A1-Pad28)") (pinfunction "~{RESET}") (pintype "input"))
@@
       (net 4 "/GND") (pinfunction "GND") (pintype "power_in"))
     (pad "30" thru_hole oval locked (at 15.24 0 270) (size 1.6 1.6) (drill 1) (layers *.Cu *.Mask)
-      (net 29 "Net-(A1-Pad30)") (pinfunction "VIN") (pintype "power_in"))
+      (net 29 "unconnected-(A1-Pad30)") (pinfunction "VIN") (pintype "power_in+no_connect"))
     (model "${KICAD6_3DMODEL_DIR}/Module.3dshapes/Arduino_Nano_WithMountingHoles.wrl"
       (offset (xyz 0 0 0))
@@
     (style (thickness 0.15) (arrow_length 1.27) (text_position_mode 0) (extension_height 0.58642) (extension_offset 0.5) keep_text_aligned)
   )
-  (segment (start 112.395 44.45) (end 111.76 43.815) (width 0.8) (layer "F.Cu") (net 4))
-  (segment (start 112.395 46.99) (end 112.395 44.45) (width 0.8) (layer "F.Cu") (net 4))
-  (segment (start 109.855 40.005) (end 111.76 38.1) (width 0.8) (layer "F.Cu") (net 4))
-  (segment (start 111.76 38.1) (end 133.985 38.1) (width 0.8) (layer "F.Cu") (net 4))
   (via (at 109.855 40.005) (size 1.85) (drill 0.8) (layers "F.Cu" "B.Cu") (net 4))
   (via (at 111.76 43.815) (size 1.85) (drill 0.8) (layers "F.Cu" "B.Cu") (net 4))
@@
   (segment (start 153.035 43.18) (end 146.685 49.53) (width 0.8) (layer "F.Cu") (net 14))
   (segment (start 146.685 49.53) (end 112.395 49.53) (width 0.8) (layer "F.Cu") (net 14))
-  (segment (start 155.575 43.18) (end 147.955 50.8) (width 0.8) (layer "F.Cu") (net 15))
+  (segment (start 147.32 51.435) (end 118.127196 51.435) (width 0.8) (layer "F.Cu") (net 15))
   (segment (start 111.125011 56.515011) (end 109.855 55.245) (width 0.8) (layer "F.Cu") (net 15))
-  (segment (start 118.762196 50.8) (end 113.047185 56.515011) (width 0.8) (layer "F.Cu") (net 15))
   (segment (start 113.047185 56.515011) (end 111.125011 56.515011) (width 0.8) (layer "F.Cu") (net 15))
-  (segment (start 147.955 50.8) (end 118.762196 50.8) (width 0.8) (layer "F.Cu") (net 15))
+  (segment (start 118.127196 51.435) (end 113.047185 56.515011) (width 0.8) (layer "F.Cu") (net 15))
   (segment (start 109.855 55.245) (end 109.855 52.07) (width 0.8) (layer "F.Cu") (net 15))
+  (segment (start 155.575 43.18) (end 147.32 51.435) (width 0.8) (layer "F.Cu") (net 15))
   (segment (start 135.128 60.96) (end 128.524 67.564) (width 0.8) (layer "F.Cu") (net 16))
   (segment (start 107.696 50.48692) (end 108.65292 49.53) (width 0.8) (layer "F.Cu") (net 16))
@@
   (segment (start 155.575 58.42) (end 153.035 60.96) (width 0.8) (layer "F.Cu") (net 16))
   (segment (start 107.696 59.436) (end 107.696 50.48692) (width 0.8) (layer "F.Cu") (net 16))
+  (segment (start 123.19 53.975) (end 127.635 58.42) (width 0.8) (layer "F.Cu") (net 27))
+  (segment (start 113.727495 58.357505) (end 118.11 53.975) (width 0.8) (layer "F.Cu") (net 27))
+  (segment (start 113.727495 58.357505) (end 112.395 58.357505) (width 0.8) (layer "F.Cu") (net 27))
+  (segment (start 112.395 54.61) (end 112.395 52.07) (width 0.8) (layer "F.Cu") (net 27))
+  (segment (start 118.11 53.975) (end 123.19 53.975) (width 0.8) (layer "F.Cu") (net 27))
+  (via (at 112.395 54.61) (size 1.85) (drill 0.8) (layers "F.Cu" "B.Cu") (net 27))
+  (via (at 112.395 58.357505) (size 1.85) (drill 0.8) (layers "F.Cu" "B.Cu") (net 27))
+  (segment (start 112.395 54.61) (end 112.395 58.357505) (width 0.8) (layer "B.Cu") (net 27))
   (segment (start 125.095 60.838) (end 127 62.743) (width 0.8) (layer "F.Cu") (net 28))
   (segment (start 125.095 58.42) (end 125.095 60.838) (width 0.8) (layer "F.Cu") (net 28))
-  (segment (start 112.519989 58.42) (end 120.015 58.42) (width 0.8) (layer "F.Cu") (net 29))
-  (segment (start 112.395 54.9405) (end 112.395 54.61) (width 0.8) (layer "F.Cu") (net 29))
-  (segment (start 112.395 54.61) (end 112.395 52.07) (width 0.8) (layer "F.Cu") (net 29))
-  (segment (start 112.395 58.295011) (end 112.395 58.357505) (width 0.8) (layer "F.Cu") (net 29))
-  (segment (start 112.395 58.357505) (end 112.519989 58.42) (width 0.8) (layer "F.Cu") (net 29))
-  (via (at 112.395 54.61) (size 1.85) (drill 0.8) (layers "F.Cu" "B.Cu") (net 29))
-  (via (at 112.395 58.357505) (size 1.85) (drill 0.8) (layers "F.Cu" "B.Cu") (net 29))
-  (segment (start 112.395 58.357505) (end 112.395 54.61) (width 0.8) (layer "B.Cu") (net 29))
   (segment (start 146.685 29.21) (end 153.035 35.56) (width 0.8) (layer "F.Cu") (net 30))
   (segment (start 116.84 29.21) (end 146.685 29.21) (width 0.8) (layer "F.Cu") (net 30))
@@
   (segment (start 130.81 32.385) (end 126.365 32.385) (width 0.8) (layer "F.Cu") (net 32))
   (segment (start 133.985 35.56) (end 130.81 32.385) (width 0.8) (layer "F.Cu") (net 32))
-  (segment (start 119.907888 65.283) (end 119.888 65.302888) (width 0.8) (layer "F.Cu") (net 33))
-  (segment (start 119.38 65.283) (end 127 65.283) (width 0.8) (layer "F.Cu") (net 33))
+  (segment (start 127 65.283) (end 119.38 65.283) (width 0.8) (layer "F.Cu") (net 33))
   (zone (net 4) (net_name "/GND") (layer "F.Cu") (hatch edge 0.508)
     (connect_pads (clearance 0.508))
